Commit message: fixed rotation and added blender script

File: src/urdf_visualize/urdf/robot copy 2.urdf (robot description, URDF)
Before this commit: robot onshape, 2 links, 0 joints
Links:
- removed link base_link
- added link compact_excavator_frame_body, mass 459.11707598787205598; collision mesh filename=package://urdf_visualize/meshes/compact_excavator_frame_bod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; visual mesh filename=package://urdf_visualize/meshes/compact_excavator_frame_bod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
- added link compact_excavator_front_wheel, mass 17.64673591392957519; collision mesh filename=package://urdf_visualize/meshes/compact_excavator_front_whe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; visual mesh filename=package://urdf_visualize/meshes/compact_excavator_front_whe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
- added link compact_excavator_front_wheel_2, mass 17.64673591392957519; collision mesh filename=package://urdf_visualize/meshes/compact_excavator_front_whe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; visual mesh filename=package://urdf_visualize/meshes/compact_excavator_front_whe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
- added link compact_excavator_main_drive_wheel_cmpl, mass 35.986291345795820007; collision mesh filename=package://urdf_visualize/meshes/compact_excavator_main_driv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; visual mesh filename=package://urdf_visualize/meshes/compact_excavator_main_driv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
- added link compact_excavator_main_drive_wheel_cmpl_(1), mass 35.986291345795820007; collision mesh filename=package://urdf_visualize/meshes/compact_excavator_main_driv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; visual mesh filename=package://urdf_visualize/meshes/compact_excavator_main_driv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
- added link compact_excavator_turret_cabin_roller, mass 72.827596459303620691; collision mesh filename=package://urdf_visualize/meshes/compact_excavator_turret_ca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; visual mesh filename=package://urdf_visualize/meshes/compact_excavator_turret_ca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
- added link part01_pin_1, mass 98.140190062279060612; collision mesh filename=package://urdf_visualize/meshes/part01_pin_1.stl; visual mesh filename=package://urdf_visualize/meshes/part01_pin_1.stl
- added link part02_cmpl, mass 694.17793513858055121; collision mesh filename=package://urdf_visualize/meshes/part02.stl; visual mesh filename=package://urdf_visualize/meshes/part02.stl
- added link part03, mass 265.34907807560875881; collision mesh filename=package://urdf_visualize/meshes/part03.stl; visual mesh filename=package://urdf_visualize/meshes/part03.stl
- added link part04, mass 132.70765933863819441; collision mesh filename=package://urdf_visualize/meshes/bucket.stl; collision mesh filename=package://urdf_visualize/meshes/bucket_mount.stl
- added link push_blade_bucket, mass 147.01808168083425699; collision mesh filename=package://urdf_visualize/meshes/push_blade_bucket.stl; visual mesh filename=package://urdf_visualize/meshes/push_blade_bucket.stl
Joints:
- added joint fixed_base: type fixed, parent compact_excavator_cabin_body_cmpl, child compact_excavator_turret_cabin_roller, origin xyz=-0.25 -2.394831672112794725e-15 0.049999999999999988898 rpy=-6.5400986663891116335e-25 -1.0029564927205460558e-23 3.1415926535897926719, axis 0 0 1, limit effort=1 velocity=20
- added joint full_arm_rotation: type revolute, parent compact_excavator_cabin_body_cmpl, child part01_pin_1, origin xyz=-0.040707723917193447405 -0.80673603465099630316 0.38039999999999996039 rpy=3.141592653589793116 4.8797124238540929311e-17 0.21446312817660284633, axis 0 0 1, limit lower=-1 upper=1.57 effort=1 velocity=20
- added joint left_idle_passive_wheel: type continuous, parent compact_excavator_frame_body, child compact_excavator_front_wheel, origin xyz=-0.61299999999999998934 0.80000000000000026645 -0.2750000000000000222 rpy=1.570796326794896558 -1.0222876983448163646 -1.5707963267948941155, axis 0 0 1, limit effort=1 velocity=20
- added joint left_sprocket_wheel: type continuous, parent compact_excavator_frame_body, child compact_excavator_main_drive_wheel_cmpl_(1), origin xyz=-0.5739999999999999547 -0.80000000000000015543 -0.2750000000000000222 rpy=1.570796326794896558 -0.3547477759675310427 1.5707963267948976682, axis 0 0 1, limit effort=1 velocity=20
- added joint lower_arm: type revolute, parent part01_pin_1, child part02_cmpl, origin xyz=0.079999999999996157518 0.074999999999997291056 -0.1500000000000039635 rpy=-1.570796326794896558 0.39285813115170314935 -1.5707963267949009989, axis 0 0 1, limit lower=-0.4 upper=0.4 effort=1 velocity=20
- added joint plow1: type revolute, parent compact_excavator_frame_body, child push_blade_bucket, origin xyz=-0.25500000000000005995 0.4880000000000002669 -0.20500000000000001554 rpy=1.570796326794896558 -1.3195606112546109934 -1.57079632679489678, axis 0 0 1, limit effort=1 velocity=20
- added joint right_idle_passive_wheel: type continuous, parent compact_excavator_frame_body, child compact_excavator_front_wheel_2, origin xyz=0.54800000000000004263 0.80000000000000015543 -0.27499999999999996669 rpy=1.57079632679489678 -1.1102232252180887662e-16 -1.5707963267948976682, axis 0 0 1, limit effort=1 velocity=20
- added joint right_sprocket_wheel: type continuous, parent compact_excavator_frame_body, child compact_excavator_main_drive_wheel_cmpl, origin xyz=0.5739999999999999547 -0.80000000000000004441 -0.2750000000000000222 rpy=1.570796326794896558 -1.2984776443375001254 -1.5707963267948972241, axis 0 0 1, limit effort=1 velocity=20
- added joint scoop1: type revolute, parent part03, child part04, origin xyz=0.12000000000000410338 -1.5403327562575612752 9.4368957093138305936e-16 rpy=3.1415926535897917837 1.8859935444767496044e-16 -1.5963552846072552871, axis 0 0 1, limit lower=-1.2217304763960306069 upper=0.87266462599716476678 effort=1 velocity=20
- added joint tankSpin_wheel: type continuous, parent compact_excavator_turret_cabin_roller, child compact_excavator_frame_body, origin xyz=-0.25 -2.6052883279480892481e-15 -0.050000000000000002776 rpy=-5.5511151231419568159e-17 -1.1102230246202266528e-16 1.57079632679489678, axis 0 0 1, limit effort=1 velocity=20
- added joint upperToLow: type revolute, parent part02_cmpl, child part03, origin xyz=-0.84000000000000030198 2.3549999999999999822 -0.13500000000000003664 rpy=3.1415926535897922278 6.9325343981756730312e-15 2.5555644018935783635, axis 0 0 1, limit lower=-0.5 upper=1.57 effort=1 velocity=20

File: src/urdf_visualize/urdf/robot.urdf (robot description, URDF)
Before this commit: robot onshape, 3 links, 2 joints
Links:
- added link compact_excavator_frame_body, mass 459.11707598787205598; collision mesh filename=package://urdf_visualize/meshes/compact_excavator_frame_bod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; visual mesh filename=package://urdf_visualize/meshes/compact_excavator_frame_bod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
- added link compact_excavator_front_wheel, mass 17.64673591392957519; collision mesh filename=package://urdf_visualize/meshes/compact_excavator_front_whe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; visual mesh filename=package://urdf_visualize/meshes/compact_excavator_front_whe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
- added link compact_excavator_front_wheel_2, mass 17.64673591392957519; collision mesh filename=package://urdf_visualize/meshes/compact_excavator_front_whe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; visual mesh filename=package://urdf_visualize/meshes/compact_excavator_front_whe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
- added link compact_excavator_main_drive_wheel_cmpl, mass 35.986291345795820007; collision mesh filename=package://urdf_visualize/meshes/compact_excavator_main_driv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; visual mesh filename=package://urdf_visualize/meshes/compact_excavator_main_driv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
- added link compact_excavator_main_drive_wheel_cmpl_(1), mass 35.986291345795820007; collision mesh filename=package://urdf_visualize/meshes/compact_excavator_main_driv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; visual mesh filename=package://urdf_visualize/meshes/compact_excavator_main_driv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
- added link compact_excavator_turret_cabin_roller, mass 72.827596459303620691; collision mesh filename=package://urdf_visualize/meshes/compact_excavator_turret_ca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; visual mesh filename=package://urdf_visualize/meshes/compact_excavator_turret_ca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
- added link part02_cmpl, mass 694.17793513858055121; collision mesh filename=package://urdf_visualize/meshes/part02.stl; visual mesh filename=package://urdf_visualize/meshes/part02.stl
- added link part03, mass 265.34907807560875881; collision mesh filename=package://urdf_visualize/meshes/part03.stl; visual mesh filename=package://urdf_visualize/meshes/part03.stl
- added link part04, mass 132.70765933863819441; collision mesh filename=package://urdf_visualize/meshes/bucket.stl; collision mesh filename=package://urdf_visualize/meshes/bucket_mount.stl
- added link push_blade_bucket, mass 147.01808168083425699; collision mesh filename=package://urdf_visualize/meshes/push_blade_bucket.stl; visual mesh filename=package://urdf_visualize/meshes/push_blade_bucket.stl
- added link world
Joints:
- added joint fixed_base: type fixed, parent compact_excavator_cabin_body_cmpl, child compact_excavator_turret_cabin_roller, origin xyz=-0.25 -2.394831672112794725e-15 0.049999999999999988898 rpy=-6.5400986663891116335e-25 -1.0029564927205460558e-23 3.1415926535897926719, axis 0 0 1, limit effort=1 velocity=20
- added joint left_idle_passive_wheel: type continuous, parent compact_excavator_frame_body, child compact_excavator_front_wheel, origin xyz=-0.61299999999999998934 0.80000000000000026645 -0.2750000000000000222 rpy=1.570796326794896558 -1.0222876983448163646 -1.5707963267948941155, axis 0 0 1, limit effort=1 velocity=20
- added joint left_sprocket_wheel: type continuous, parent compact_excavator_frame_body, child compact_excavator_main_drive_wheel_cmpl_(1), origin xyz=-0.5739999999999999547 -0.80000000000000015543 -0.2750000000000000222 rpy=1.570796326794896558 -0.3547477759675310427 1.5707963267948976682, axis 0 0 1, limit effort=1 velocity=20
- added joint lower_arm: type revolute, parent part01_pin_1, child part02_cmpl, origin xyz=0.079999999999996157518 0.074999999999997291056 -0.1500000000000039635 rpy=-1.570796326794896558 0.39285813115170314935 -1.5707963267949009989, axis 0 0 1, limit lower=-0.4 upper=0.4 effort=1 velocity=20
- added joint plow1: type revolute, parent compact_excavator_frame_body, child push_blade_bucket, origin xyz=-0.25500000000000005995 0.4880000000000002669 -0.20500000000000001554 rpy=1.570796326794896558 -1.3195606112546109934 -1.57079632679489678, axis 0 0 1, limit effort=1 velocity=20
- added joint right_idle_passive_wheel: type continuous, parent compact_excavator_frame_body, child compact_excavator_front_wheel_2, origin xyz=0.54800000000000004263 0.80000000000000015543 -0.27499999999999996669 rpy=1.57079632679489678 -1.1102232252180887662e-16 -1.5707963267948976682, axis 0 0 1, limit effort=1 velocity=20
- added joint right_sprocket_wheel: type continuous, parent compact_excavator_frame_body, child compact_excavator_main_drive_wheel_cmpl, origin xyz=0.5739999999999999547 -0.80000000000000004441 -0.2750000000000000222 rpy=1.570796326794896558 -1.2984776443375001254 -1.5707963267948972241, axis 0 0 1, limit effort=1 velocity=20
- added joint scoop1: type revolute, parent part03, child part04, origin xyz=0.12000000000000410338 -1.5403327562575612752 9.4368957093138305936e-16 rpy=3.1415926535897917837 1.8859935444767496044e-16 -1.5963552846072552871, axis 0 0 1, limit lower=-1.2217304763960306069 upper=0.87266462599716476678 effort=1 velocity=20
- added joint tankSpin_wheel: type continuous, parent compact_excavator_turret_cabin_roller, child compact_excavator_frame_body, origin xyz=-0.25 -2.6052883279480892481e-15 -0.050000000000000002776 rpy=-5.5511151231419568159e-17 -1.1102230246202266528e-16 1.57079632679489678, axis 0 0 1, limit effort=1 velocity=20
- added joint upperToLow: type revolute, parent part02_cmpl, child part03, origin xyz=-0.84000000000000030198 2.3549999999999999822 -0.13500000000000003664 rpy=3.1415926535897922278 6.9325343981756730312e-15 2.5555644018935783635, axis 0 0 1, limit lower=-0.5 upper=1.57 effort=1 velocity=20
- added joint world_to_base: type fixed, parent world, child base_link, origin xyz=0 0 0 rpy=-1.5708 0 0
- joint base_to_cabin: origin xyz=0.15929227608280682738 -0.2512819772778476235 0.33139999999999991687 rpy=1.5707 0 0 -> xyz=0.15929227608280682738 -0.2512819772778476235 0.33139999999999991687 rpy=0 0 0
- joint full_arm_rotation: origin xyz=-0.040707723917193447405 -0.80673603465099630316 0.38039999999999996039 rpy=3.14159 0 0.2144 -> xyz=-0.040707723917193447405 -0.80673603465099630316 0.38039999999999996039 rpy=3.141592653589793116 4.8797124238540929311e-17 0.21446312817660284633
