Commit message: fixed plow

File: src/urdf_visualize/urdf/robot copy.urdf (robot description, URDF)
Before this commit: robot onshape, 12 links, 11 joints
Links:
- added link base_link
- added link world
Joints:
- added joint base_to_cabin: type fixed, parent base_link, child compact_excavator_cabin_body_cmpl, origin xyz=0.15929227608280682738 -0.2512819772778476235 0.33139999999999991687 rpy=0 0 0, axis 0 0 1
- added joint world_to_base: type fixed, parent world, child base_link, origin xyz=0 0 0 rpy=-1.5708 0 0

File: src/urdf_visualize/urdf/robot.urdf (robot description, URDF)
Before this commit: robot onshape, 14 links, 13 joints
Joints:
- joint plow1: limit effort=1 velocity=20 -> lower=0.2 upper=0 effort=1 velocity=20

Commit message: cleanup and fixing visual and collision origins

File: src/urdf_visualize/urdf/robot copy.urdf (robot description, URDF)
Before this commit: robot onshape, 14 links, 13 joints
Joints:
- joint plow1: limit effort=1 velocity=20 -> lower=0.2 upper=0 effort=1 velocity=20
- joint world_to_base: origin xyz=0 0 0 rpy=-1.5708 0 0 -> xyz=10 10 0 rpy=0 0 0

File: src/urdf_visualize/urdf/robot.urdf (robot description, URDF)
Before this commit: robot onshape, 14 links, 13 joints
Joints:
- joint tankSpin_wheel: origin xyz=-0.25 -2.6052883279480892481e-15 -0.050000000000000002776 rpy=-5.5511151231419568159e-17 -1.1102230246202266528e-16 1.57079632679489678 -> xyz=-0.25 -2.6052883279480892481e-15 -0.050000000000000002776 rpy=-5.5511151231419568159e-17 -1.1102230246202266528e-16 0
- joint world_to_base: origin xyz=0 0 0 rpy=-1.5708 0 0 -> xyz=3 3 0 rpy=0 0 0
