Commit message: changed name

File: src/urdf_visualize/urdf/robot.urdf (robot description, URDF)
Before this commit: robot onshape, 14 links, 13 joints
Links:
- removed link compact_excavator_cabin_body_cmpl
- removed link compact_excavator_frame_body
- removed link compact_excavator_front_wheel
- removed link compact_excavator_front_wheel_2
- removed link compact_excavator_main_drive_wheel_cmpl
- removed link compact_excavator_main_drive_wheel_cmpl_(1)
- removed link part01_pin_1
- removed link part02_cmpl
- removed link part03
- removed link part04
- added link arm_base, mass 265.34907807560875881; collision mesh filename=package://urdf_visualize/meshes/part03.stl; visual mesh filename=package://urdf_visualize/meshes/part03.stl
- added link boom_base, mass 694.17793513858055121; collision mesh filename=package://urdf_visualize/meshes/part02.stl; visual mesh filename=package://urdf_visualize/meshes/part02.stl
- added link bucket_base, mass 132.70765933863819441; collision mesh filename=package://urdf_visualize/meshes/bucket.stl; collision mesh filename=package://urdf_visualize/meshes/bucket_mount.stl
- added link cabin_base, mass 9732.8038980797628028; collision mesh filename=package://urdf_visualize/meshes/compact_excavator_cabin_bod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; visual mesh filename=package://urdf_visualize/meshes/compact_excavator_cabin_bod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
- added link left_front_wheel_link, mass 17.64673591392957519; collision mesh filename=package://urdf_visualize/meshes/compact_excavator_front_whe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; visual mesh filename=package://urdf_visualize/meshes/compact_excavator_front_whe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
- added link left_spining_wheel_link, mass 35.986291345795820007; collision mesh filename=package://urdf_visualize/meshes/compact_excavator_main_driv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; visual mesh filename=package://urdf_visualize/meshes/compact_excavator_main_driv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
- added link right_front_wheel_link, mass 17.64673591392957519; collision mesh filename=package://urdf_visualize/meshes/compact_excavator_front_whe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; visual mesh filename=package://urdf_visualize/meshes/compact_excavator_front_whe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
- added link right_spinning_wheel_link, mass 35.986291345795820007; collision mesh filename=package://urdf_visualize/meshes/compact_excavator_main_driv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; visual mesh filename=package://urdf_visualize/meshes/compact_excavator_main_driv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
- added link swing_base, mass 98.140190062279060612; collision mesh filename=package://urdf_visualize/meshes/part01_pin_1.stl; visual mesh filename=package://urdf_visualize/meshes/part01_pin_1.stl
- added link turret_base, mass 459.11707598787205598; collision mesh filename=package://urdf_visualize/meshes/compact_excavator_frame_bod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; visual mesh filename=package://urdf_visualize/meshes/compact_excavator_frame_bod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
Joints:
- removed joint left_sprocket_wheel
- added joint left_spining_wheel: type continuous, parent turret_base, child left_spining_wheel_link, origin xyz=-0.5739999999999999547 -0.80000000000000015543 -0.2750000000000000222 rpy=1.570796326794896558 -0.3547477759675310427 1.5707963267948976682, axis 0 0 1, limit effort=1 velocity=20
- joint base_to_cabin: child compact_excavator_cabin_body_cmpl -> cabin_base
- joint fixed_base: parent compact_excavator_cabin_body_cmpl -> cabin_base
- joint full_arm_rotation: child part01_pin_1 -> swing_base; parent compact_excavator_cabin_body_cmpl -> cabin_base
- joint left_idle_passive_wheel: child compact_excavator_front_wheel -> left_front_wheel_link; parent compact_excavator_frame_body -> turret_base
- joint lower_arm: child part02_cmpl -> boom_base; parent part01_pin_1 -> swing_base
- joint plow1: parent compact_excavator_frame_body -> turret_base
- joint right_idle_passive_wheel: child compact_excavator_front_wheel_2 -> right_front_wheel_link; parent compact_excavator_frame_body -> turret_base
- joint right_sprocket_wheel: child compact_excavator_main_drive_wheel_cmpl -> right_spinning_wheel_link; parent compact_excavator_frame_body -> turret_base
- joint scoop1: child part04 -> bucket_base; parent part03 -> arm_base
- joint tankSpin_wheel: child compact_excavator_frame_body -> turret_base
- joint upperToLow: child part03 -> arm_base; parent part02_cmpl -> boom_base

Commit message: fixed joint names

File: src/urdf_visualize/urdf/robot.urdf (robot description, URDF)
Before this commit: robot onshape, 14 links, 13 joints
Links:
- removed link left_spining_wheel_link
- added link left_spinning_wheel_link, mass 35.986291345795820007; collision mesh filename=package://urdf_visualize/meshes/compact_excavator_main_driv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; visual mesh filename=package://urdf_visualize/meshes/compact_excavator_main_driv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
Joints:
- removed joint full_arm_rotation
- removed joint left_idle_passive_wheel
- removed joint left_spining_wheel
- removed joint lower_arm
- removed joint plow1
- removed joint right_idle_passive_wheel
- removed joint right_sprocket_wheel
- removed joint scoop1
- removed joint tankSpin_wheel
- removed joint upperToLow
- added joint arm_to_boom: type revolute, parent boom_base, child arm_base, origin xyz=-0.84000000000000030198 2.3549999999999999822 -0.13500000000000003664 rpy=3.1415926535897922278 6.9325343981756730312e-15 2.5555644018935783635, axis 0 0 1, limit lower=-0.5 upper=1.57 effort=1 velocity=20
- added joint boom_to_swing: type revolute, parent swing_base, child boom_base, origin xyz=0.079999999999996157518 0.074999999999997291056 -0.1500000000000039635 rpy=-1.570796326794896558 0.39285813115170314935 -1.5707963267949009989, axis 0 0 1, limit lower=-0.4 upper=0.4 effort=1 velocity=20
- added joint bucket_to_arm: type revolute, parent arm_base, child bucket_base, origin xyz=0.12000000000000410338 -1.5403327562575612752 9.4368957093138305936e-16 rpy=3.1415926535897917837 1.8859935444767496044e-16 -1.5963552846072552871, axis 0 0 1, limit lower=-1.2217304763960306069 upper=0.87266462599716476678 effort=1 velocity=20
- added joint left_passive_wheel: type continuous, parent turret_base, child left_front_wheel_link, origin xyz=-0.61299999999999998934 0.80000000000000026645 -0.2750000000000000222 rpy=1.570796326794896558 -1.0222876983448163646 -1.5707963267948941155, axis 0 0 1, limit effort=1 velocity=20
- added joint left_spinning_wheel: type continuous, parent turret_base, child left_spinning_wheel_link, origin xyz=-0.5739999999999999547 -0.80000000000000015543 -0.2750000000000000222 rpy=1.570796326794896558 -0.3547477759675310427 1.5707963267948976682, axis 0 0 1, limit effort=1 velocity=20
- added joint plow_to_base: type revolute, parent turret_base, child push_blade_bucket, origin xyz=-0.25500000000000005995 0.4880000000000002669 -0.20500000000000001554 rpy=1.570796326794896558 -1.3195606112546109934 -1.57079632679489678, axis 0 0 1, limit lower=0.2 upper=0 effort=1 velocity=20
- added joint right_passive_wheel: type continuous, parent turret_base, child right_front_wheel_link, origin xyz=0.54800000000000004263 0.80000000000000015543 -0.27499999999999996669 rpy=1.57079632679489678 -1.1102232252180887662e-16 -1.5707963267948976682, axis 0 0 1, limit effort=1 velocity=20
- added joint right_spinning_wheel: type continuous, parent turret_base, child right_spinning_wheel_link, origin xyz=0.5739999999999999547 -0.80000000000000004441 -0.2750000000000000222 rpy=1.570796326794896558 -1.2984776443375001254 -1.5707963267948972241, axis 0 0 1, limit effort=1 velocity=20
- added joint slew: type continuous, parent compact_excavator_turret_cabin_roller, child turret_base, origin xyz=-0.25 -2.6052883279480892481e-15 -0.050000000000000002776 rpy=-5.5511151231419568159e-17 -1.1102230246202266528e-16 0, axis 0 0 1, limit effort=1 velocity=20
- added joint swing_to_cabin: type revolute, parent cabin_base, child swing_base, origin xyz=-0.040707723917193447405 -0.80673603465099630316 0.38039999999999996039 rpy=3.141592653589793116 4.8797124238540929311e-17 0.21446312817660284633, axis 0 0 1, limit lower=-1 upper=1.57 effort=1 velocity=20

Commit message: pre joint fix

File: src/urdf_visualize/urdf/robot.urdf (robot description, URDF)
Before this commit: robot onshape, 14 links, 13 joints
Joints:
- joint world_to_base: origin xyz=3 3 0 rpy=0 0 0 -> xyz=0 0 0 rpy=0 0 0

Commit message: probably fixed the slew problem

File: src/urdf_visualize/urdf/robot.urdf (robot description, URDF)
Before this commit: robot onshape, 14 links, 13 joints
Links:
- removed link compact_excavator_turret_cabin_roller
Joints:
- removed joint base_to_cabin
- removed joint fixed_base
- removed joint world_to_base
- added joint base_to_turret: type fixed, parent base_link, child turret_base, origin xyz=0 0 0.45 rpy=0 0 0, axis 0 0 1
- added joint world_to_base_link: type fixed, parent world, child base_link, origin xyz=0 0 0 rpy=0 0 0
- joint slew: child turret_base -> cabin_base; origin xyz=-0.25 -2.6052883279480892481e-15 -0.050000000000000002776 rpy=-5.5511151231419568159e-17 -1.1102230246202266528e-16 0 -> xyz=0 0 0 rpy=-5.5511151231419568159e-17 -1.1102230246202266528e-16 -3.1415; parent compact_excavator_turret_cabin_roller -> turret_base

Commit message: trying xacro

File: src/urdf_visualize/urdf/robot.urdf (robot description, URDF)
Before this commit: robot onshape, 13 links, 12 joints
Links:
- link cabin_base: mass 9732.8038980797628028 -> 9732.8039
- link turret_base: mass 459.11707598787205598 -> 459.1171

Commit message: trying gazebo spawn

File: src/urdf_visualize/urdf/robot.urdf (robot description, URDF)
Before this commit: robot onshape, 13 links, 12 joints
Links:
- added link wheel_left_free, mass 43.19562500000001; collision cylinder length=0.2 radius=0.25; visual cylinder length=0.2 radius=0.25
- added link wheel_left_spinning, mass 43.19562500000001; collision cylinder length=0.2 radius=0.25; visual cylinder length=0.2 radius=0.25
- added link wheel_right_free, mass 43.19562500000001; collision cylinder length=0.2 radius=0.25; visual cylinder length=0.2 radius=0.25
- added link wheel_right_spinning, mass 43.19562500000001; collision cylinder length=0.2 radius=0.25; visual cylinder length=0.2 radius=0.25
Joints:
- added joint left_passive_wheel_joint: type continuous, parent left_front_wheel_link, child wheel_left_free, origin xyz=0 0 0.3 rpy=0 0 0, axis 0 0 1, limit effort=1 velocity=20
- added joint left_spinning_wheel_joint: type continuous, parent left_spinning_wheel_link, child wheel_left_spinning, origin xyz=0 0 -0.3 rpy=0 0 0, axis 0 0 1, limit effort=1 velocity=20
- added joint right_passive_wheel_joint: type continuous, parent right_front_wheel_link, child wheel_right_free, origin xyz=0 0 -0.3 rpy=0 0 0, axis 0 0 1, limit effort=1 velocity=20
- added joint right_spinning_wheel_joint: type continuous, parent right_spinning_wheel_link, child wheel_right_spinning, origin xyz=0 0 -0.3 rpy=0 0 0, axis 0 0 1, limit effort=1 velocity=20
- joint base_to_turret: origin xyz=0 0 0.45 rpy=0 0 0 -> xyz=0 0 0.55 rpy=0 0 0

Commit message: removed world link to test gravity

File: src/urdf_visualize/urdf/robot.urdf (robot description, URDF)
Before this commit: robot onshape, 17 links, 16 joints
Links:
- removed link world
Joints:
- removed joint world_to_base_link

File: src/urdf_visualize/urdf/robot_wheel.xacro (robot description, xacro)
@@ -1,5 +1,5 @@
 <?xml version="1.0"?>
 <robot xmlns:xacro="http://www.ros.org/wiki/xacro" name="onshape">
-    <link name="world"/>
+    <!-- <link name="world"/> -->
     <xacro:property name="mesh_root" value="package://urdf_visualize/meshes"/>
     <xacro:property name="cabin_base_mesh" value="${mesh_root}/compact_excavator_cabin_body.stl"/>
@@ -441,9 +441,9 @@
         <joint_properties friction="0.0"/>
     </joint>
-    <joint name="world_to_base_link" type="fixed">
+    <!-- <joint name="world_to_base_link" type="fixed">
         <parent link="world"/>
         <child link="base_link"/>
         <origin xyz="0 0 0" rpy="0 0 0"/>
-    </joint>
+    </joint> -->
     <joint name="base_to_turret" type="fixed">
         <origin xyz="0 0 0.55" rpy="0 0 0" />
@@ -561,4 +561,5 @@
         <joint_properties friction="0.0"/>
     </joint>
+    <gravity>1</gravity>
     <ros2_control name="GazeboSystem" type="system">
         <hardware>
